File: ThreeToOne/ThreeToOne.sch (KiCad schematic (older format))
At the start: 204 parts, among them SW1 Switch, SW10 Switch, SW100 Switch, SW101 Switch, SW11 Switch, SW12 Switch, SW13 Switch, SW14 Switch, SW15 Switch, SW16 Switch, SW17 REsw, SW18 Switch, SW19 Switch, SW2 Switch, SW20 Switch, SW21 Switch, SW22 Switch, SW23 Switch, SW24 Switch, SW25 Switch, SW26 Switch, SW27 Switch, SW28 Switch, SW29 Switch, SW3 Switch, SW30 Switch, SW31 Switch, SW32 Switch, SW33 Switch, SW34 Switch, SW35 Switch, SW36 Switch, SW37 Switch, SW38 Switch, SW39 Switch, SW4 Switch, SW40 Switch, SW41 Switch, SW42 Switch, SW43 Switch, SW44 Switch, SW45 Switch, SW46 Switch, SW47 Switch, SW48 Switch, SW49 Switch, SW5 Switch, SW50 Switch, SW51 Switch, SW52 Switch, SW53 Switch, SW54 Switch, SW55 Switch, SW56 Switch, SW57 Switch, SW58 Switch, SW59 Switch, SW6 Switch, SW60 Switch, SW61 Switch, SW62 Switch, SW63 Switch, SW64 Switch, SW65 Switch, SW66 Switch, SW67 Switch, SW68 Switch, SW69 Switch, SW7 Switch, SW70 Switch, SW71 Switch, SW72 Switch, SW73 Switch, SW74 Switch, SW75 Switch, SW76 Switch, SW77 Switch, SW78 Switch, SW79 Switch, SW8 Switch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

Commit message: Assigned footprints
Parts:
- added H1, H10, H11, H12, H2, H3, H4, H5, H6, H7, H8, H9: Hole, symbol KeyboardLibrary:Hole
- D1, D10, D100, D101, D11, D12, D13, D14, D15, D16, D17, D18, D19, D2, D20, D21, D22, D23, D24, D25, D26, D27, D28, D29, D3, D30, D31, D32, D33, D34, D35, D36, D37, D38, D39, D4, D40, D41, D42, D43, D44, D45, D46, D47, D48, D49, D5, D50, D51, D52, D53, D54, D55, D56, D57, D58, D59, D6, D60, D61, D62, D63, D64, D65, D66, D67, D68, D69, D7, D70, D71, D72, D73, D74, D75, D76, D77, D78, D79, D8, D80, D81, D82, D83, D84, D85, D86, D87, D88, D89, D9, D90, D91, D92, D93, D94, D95, D96, D97, D98, D99: footprint (none) -> KeyboardFootprints:Diode
- SW1, SW10, SW100, SW101, SW11, SW12, SW13, SW14, SW15, SW16, SW17, SW18, SW19, SW2, SW20, SW21, SW22, SW23, SW24, SW25, SW26, SW27, SW28, SW29, SW3, SW30, SW31, SW32, SW33, SW34, SW35, SW36, SW37, SW38, SW39, SW4, SW40, SW41, SW42, SW43, SW44, SW45, SW46, SW47, SW48, SW49, SW5, SW50, SW51, SW52, SW53, SW54, SW55, SW56, SW57, SW58, SW59, SW6, SW60, SW61, SW62, SW63, SW64, SW65, SW66, SW67, SW68, SW69, SW7, SW70, SW71, SW72, SW73, SW74, SW75, SW76, SW77, SW78, SW79, SW8, SW80, SW81, SW82, SW83, SW84, SW85, SW86, SW87, SW88, SW89, SW9, SW90, SW92, SW93, SW94, SW95, SW96, SW97, SW98, SW99: footprint (none) -> KeyboardFootprints:MX_Choc_Symmetric
- SW91: footprint (none) -> KeyboardFootprints:REsw
- U1, U2: footprint (none) -> KeyboardFootprints:ProMicro
